Commit message: Created driven robot

File: description/robot_core.xacro (robot description, xacro)
@@ -1,6 +1,6 @@
 <?xml version="1.0"?>
 <robot xmlns:xacro="http://www.ros.org/wiki/xacro" >
-    <xacro:include filename="inertial_macros.xacro">
-  <material name="white">
+    <xacro:include filename="inertial_macros.xacro"/>
+    <material name="white">
         <color rgba="1 1 1 1" />
     </material>
@@ -14,19 +14,16 @@
         <color rgba="0 0 0 1"/>
     </material>
-    <material name="red">
-        <color rgba="1 0 0 1"/>
-    </material>
-     <!-- BASE LINK -->
+    <!-- BASE LINK -->
     <link name="base_link">
     </link>
-<!--CHASSIS LINK-->
-  <joint name="chassis_joint" type="fixed">
+    <!-- CHASSIS LINK -->
+    <joint name="chassis_joint" type="fixed">
         <parent link="base_link"/>
         <child link="chassis"/>
         <origin xyz="-0.1 0 0"/>
     </joint>
-    <link name="chassis_joint">
+    <link name="chassis">
         <visual>
-            <origin xyz="0.15 0 0.75"/>
+            <origin xyz="0.15 0 0.075"/>
             <geometry>
                 <box size="0.3 0.3 0.15"/>
@@ -34,6 +31,18 @@
             <material name="white"/>
         </visual>
+        <collision>
+            <origin xyz="0.15 0 0.075"/>
+            <geometry>
+                <box size="0.3 0.3 0.15"/>
+            </geometry>
+        </collision>
+        <xacro:inertial_box mass="0.5" x="0.3" y="0.3" z="0.15">
+            <origin xyz="0.15 0 0.075" rpy="0 0 0"/>
+        </xacro:inertial_box>
     </link>
-<!-- LEFT WHEEL LINK -->
+    <gazebo reference="chassis">
+        <material>Gazebo/White</material>
+    </gazebo>
+    <!-- LEFT WHEEL LINK -->
     <joint name="left_wheel_joint" type="continuous">
         <parent link="base_link"/>
@@ -42,5 +51,5 @@
         <axis xyz="0 0 1"/>
     </joint>
-  <link name="left_wheel">
+    <link name="left_wheel">
         <visual>
             <geometry>
@@ -51,8 +60,14 @@
         <collision>
             <geometry>
-                <sphere radius="0.05"/>
+                <cylinder radius="0.05" length="0.04"/>
             </geometry>
         </collision>
+        <xacro:inertial_cylinder mass="0.1" length="0.04" radius="0.05">
+            <origin xyz="0 0 0" rpy="0 0 0"/>
+        </xacro:inertial_cylinder>
     </link>
+    <gazebo reference="left_wheel">
+        <material>Gazebo/Blue</material>
+    </gazebo>
     <!-- RIGHT WHEEL LINK -->
     <joint name="right_wheel_joint" type="continuous">
@@ -71,9 +86,15 @@
         <collision>
             <geometry>
-                <sphere radius="0.05"/>
+                <cylinder radius="0.05" length="0.04"/>
             </geometry>
         </collision>
+        <xacro:inertial_cylinder mass="0.1" length="0.04" radius="0.05">
+            <origin xyz="0 0 0" rpy="0 0 0"/>
+        </xacro:inertial_cylinder>
     </link>
-     <!-- CASTER WHEEL LINK -->
+    <gazebo reference="right_wheel">
+        <material>Gazebo/Blue</material>
+    </gazebo>
+    <!-- CASTER WHEEL LINK -->
     <joint name="caster_wheel_joint" type="fixed">
         <parent link="chassis"/>
@@ -93,4 +114,12 @@
             </geometry>
         </collision>
+        <xacro:inertial_sphere mass="0.1" radius="0.05">
+            <origin xyz="0 0 0" rpy="0 0 0"/>
+        </xacro:inertial_sphere>
     </link>
+    <gazebo reference="caster_wheel">
+        <material>Gazebo/Black</material>
+        <mu1 value="0.001"/>
+        <mu2 value="0.001"/>
+    </gazebo>
 </robot>
